File: main_board.sch (EAGLE design)
At the start: 20 parts, among them IC1 AD8541RJ, T1 ATB3225

Commit message: in progress..
Parts:
- added C5: 100p, rcl:C-EUC0805
- added C6: 100n, rcl:C-EUC0805
- added C7: 10n, rcl:C-EUC0805
- added JP6: 3V3, pinhead:PINHD-1X1
- added JP7: V-OUT, pinhead:PINHD-1X1
- added JP8: GND, pinhead:PINHD-1X1
- added LX1: Ferrite bead, SignalCommunications (rev18e):WE-KI_0805A_744760022A
- added R7: 4.3k, resistor:R-EU_M0805
- added R8: 2.2M, resistor:R-EU_M0805
- added R9: 1k, resistor:R-EU_M0805
- C2: value 10u -> 10n
- C3: value 10n -> 10u
- JP1: value HV -> VCC
- JP2: value PUMP -> HV
- JP3: value TEST -> PUMP
- JP4: value VCC -> GND
- JP5: value GND -> TEST
- R1: value 22 -> 10k
- R2: value 10k -> 470
- R3: value 150k -> 22
- R4: value 4.3k -> 10k
- R5: value 470 -> 150k
- R6: value 10k -> 5.1G; device resistor:R-EU_M0805 -> resistor:R-EU_0817/22
Connections:
- new net +3V3: JP6.1, LX1.2
- new net N$10: IC1.IN-, IC1.OUT, R9.2
- new net N$11: C7.2, JP7.1, R9.1
- new net N$14: C5.2, IC1.IN+, R6.2, R8.2
- new net N$2: C6.2, IC1.+VS, LX1.1
- net GND: now also C3.2, C5.1, C6.1, C7.1, IC1.-VS, JP4.1, JP8.1, R1.1, R4.1, R7.2, R8.1; no longer C2.2, JP5.1, R2.1, R4.2, R6.1
- net HV: now also JP2.1, R6.1; no longer JP1.1
- net N$3: now also C2.1; no longer C3.1
- net N$4: now also C3.1, R3.1; no longer C2.1, R1.1
- net N$5: now also C2.2, R4.2; no longer C3.2, R2.2
- net N$7: now also R2.1; no longer R5.1
- net N$9: now also R5.2; no longer R3.2
- net PUMP: now also JP3.1, R1.2, R2.2; no longer JP2.1, R5.2, R6.2
- net TEST: now also JP5.1, R5.1, R7.1; no longer JP3.1, R3.1, R4.1
- net VCC: now also JP1.1, R3.2; no longer JP4.1, R1.2
Other:
- moved on the sheet: C2, C3, JP1, JP2, JP3, JP4, JP5, R1, R2, R3, R4, R5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

Commit message: almost completed
Parts:
- added C8: TEST, rcl:C-EUC1206
- added R10, R11, R12: 2.2M, resistor:R-EU_M0805
- JP5: value TEST -> FB
Connections:
- net N$11 renamed V-OUT
- new net FB: JP5.1, R5.1, R7.1
- new net N$6: R10.2, R11.1
- new net N$8: R11.2, R12.1
- net GND: now also C8.2
- net HV: now also R10.1
- net TEST: now also C8.1, R12.2; no longer JP5.1, R5.1, R7.1
